File: VGACard.kicad_sch (KiCad schematic)
At the start: 51 parts, among them U1 74LS161, U2 74LS161, U3 74LS161, U4 556RT4, U5 74LS161, U6 74LS161, U7 74LS161, U8 74LS10, U9 556RT4, X1 25.175MHz

Commit message: Adding timing
Parts:
- added U10: 74LS10, Package_DIP:DIP-14_W7.62mm_Socket_LongPads, symbol 74xx:74LS10
- added U11: 7400, Package_DIP:DIP-14_W7.62mm_Socket_LongPads, symbol 74xx:7400
- added U12: 74LS74, Package_DIP:DIP-14_W7.62mm_Socket_LongPads, symbol 74xx:74LS74
- added unit 3 of U8
- added unit 2 of U8
Connections:
- net +5V: now also U10.14 (VCC), U11.14 (VCC), U12.10 (~{S}), U12.14 (VCC)
- net GND: now also U10.7 (GND), U11.7 (GND), U12.2 (D), U12.3 (C), U12.7 (GND)
- net H0: now also U12.11 (C), U8.3
- net H1: now also U10.2, U8.4
- net H2: now also U8.5
- net H3: now also U11.2
- net H4: now also U10.13, U11.4, U11.5
- net H5: now also U11.1
- new net: U11.10, U11.6
- new net: U11.12, U11.8
- new net: U11.9, U8.6
- new net: U11.3, U12.4 (~{S})
- new net: U11.11, U12.13 (~{R})
- new net HBlank: U10.1, U11.13, U12.12 (D), U12.5 (Q)
- new net RESET: U8.8
- new net ~{RESET}: U10.12, U12.1 (~{R}), U8.10, U8.11, U8.9
- new net ~{SYNC}: U12.8 (~{Q})
